File: PCB/Small Edge Connector Board/DJet Small Edge Connector Board/DJet Small Edge Connector Board.sch (KiCad schematic (older format))
At the start: 27 parts, among them J1 Conn_01x01, J10 Conn_01x01, J11 Conn_01x01, J12 Conn_01x01, J13 Conn_01x01, J14 Conn_01x01, J15 Conn_01x01, J16 Conn_01x01, J17 Conn_01x01, J18 Conn_01x01, J19 Conn_01x01, J2 Conn_01x01, J20 Conn_01x01, J21 Conn_01x01, J22 Conn_01x01, J23 Conn_01x01, J24 Conn_01x01, J25 Conn_01x01, J26 Conn_01x25, J27 Conn_01x25, J3 Conn_01x01, J4 Conn_01x01, J5 Conn_01x01, J6 Conn_01x01, J7 Conn_01x01, J8 Conn_01x01, J9 Conn_01x01

Commit message: Working on updated design.
Parts:
- J1, J10, J11, J12, J13, J14, J15, J16, J17, J18, J19, J2, J20, J21, J22, J23, J24, J25, J3, J4, J5, J6, J7, J8, J9: manf# (none) -> S7121-42R
Changed lines of the file:
@@
 F 2 "Britishideas:TE-1871059-1" H 2400 2100 50  0001 C CNN
 F 3 "~" H 2400 2100 50  0001 C CNN
+F 4 "S7121-42R" H 2400 2100 50  0001 C CNN "manf#"
 	1    2400 2100
 	-1   0    0    1
@@
 F 2 "Britishideas:TE-1871059-1" H 2400 2250 50  0001 C CNN
 F 3 "~" H 2400 2250 50  0001 C CNN
+F 4 "S7121-42R" H 2400 2250 50  0001 C CNN "manf#"
 	1    2400 2250
 	-1   0    0    1
@@
 F 2 "Britishideas:TE-1871059-1" H 2400 2400 50  0001 C CNN
 F 3 "~" H 2400 2400 50  0001 C CNN
+F 4 "S7121-42R" H 2400 2400 50  0001 C CNN "manf#"
 	1    2400 2400
 	-1   0    0    1
@@
 F 2 "Britishideas:TE-1871059-1" H 2400 2550 50  0001 C CNN
 F 3 "~" H 2400 2550 50  0001 C CNN
+F 4 "S7121-42R" H 2400 2550 50  0001 C CNN "manf#"
 	1    2400 2550
 	-1   0    0    1
@@
 F 2 "Britishideas:TE-1871059-1" H 2400 2700 50  0001 C CNN
 F 3 "~" H 2400 2700 50  0001 C CNN
+F 4 "S7121-42R" H 2400 2700 50  0001 C CNN "manf#"
 	1    2400 2700
 	-1   0    0    1
@@
 F 2 "Britishideas:TE-1871059-1" H 2400 2850 50  0001 C CNN
 F 3 "~" H 2400 2850 50  0001 C CNN
+F 4 "S7121-42R" H 2400 2850 50  0001 C CNN "manf#"
 	1    2400 2850
 	-1   0    0    1
@@
 F 2 "Britishideas:TE-1871059-1" H 2400 3000 50  0001 C CNN
 F 3 "~" H 2400 3000 50  0001 C CNN
+F 4 "S7121-42R" H 2400 3000 50  0001 C CNN "manf#"
 	1    2400 3000
 	-1   0    0    1
@@
 F 2 "Britishideas:TE-1871059-1" H 2400 3150 50  0001 C CNN
 F 3 "~" H 2400 3150 50  0001 C CNN
+F 4 "S7121-42R" H 2400 3150 50  0001 C CNN "manf#"
 	1    2400 3150
 	-1   0    0    1
@@
 F 2 "Britishideas:TE-1871059-1" H 2400 3300 50  0001 C CNN
 F 3 "~" H 2400 3300 50  0001 C CNN
+F 4 "S7121-42R" H 2400 3300 50  0001 C CNN "manf#"
 	1    2400 3300
 	-1   0    0    1
@@
 F 2 "Britishideas:TE-1871059-1" H 2400 3450 50  0001 C CNN
 F 3 "~" H 2400 3450 50  0001 C CNN
+F 4 "S7121-42R" H 2400 3450 50  0001 C CNN "manf#"
 	1    2400 3450
 	-1   0    0    1
@@
 F 2 "Britishideas:TE-1871059-1" H 2400 3600 50  0001 C CNN
 F 3 "~" H 2400 3600 50  0001 C CNN
+F 4 "S7121-42R" H 2400 3600 50  0001 C CNN "manf#"
 	1    2400 3600
 	-1   0    0    1
@@
 F 2 "Britishideas:TE-1871059-1" H 2400 3750 50  0001 C CNN
 F 3 "~" H 2400 3750 50  0001 C CNN
+F 4 "S7121-42R" H 2400 3750 50  0001 C CNN "manf#"
 	1    2400 3750
 	-1   0    0    1
@@
 F 2 "Britishideas:TE-1871059-1" H 2400 3900 50  0001 C CNN
 F 3 "~" H 2400 3900 50  0001 C CNN
+F 4 "S7121-42R" H 2400 3900 50  0001 C CNN "manf#"
 	1    2400 3900
 	-1   0    0    1
@@
 F 2 "Britishideas:TE-1871059-1" H 2400 4050 50  0001 C CNN
 F 3 "~" H 2400 4050 50  0001 C CNN
+F 4 "S7121-42R" H 2400 4050 50  0001 C CNN "manf#"
 	1    2400 4050
 	-1   0    0    1
@@
 F 2 "Britishideas:TE-1871059-1" H 2400 4200 50  0001 C CNN
 F 3 "~" H 2400 4200 50  0001 C CNN
+F 4 "S7121-42R" H 2400 4200 50  0001 C CNN "manf#"
 	1    2400 4200
 	-1   0    0    1
@@
 F 2 "Britishideas:TE-1871059-1" H 2400 4350 50  0001 C CNN
 F 3 "~" H 2400 4350 50  0001 C CNN
+F 4 "S7121-42R" H 2400 4350 50  0001 C CNN "manf#"
 	1    2400 4350
 	-1   0    0    1
@@
 F 2 "Britishideas:TE-1871059-1" H 2400 4500 50  0001 C CNN
 F 3 "~" H 2400 4500 50  0001 C CNN
+F 4 "S7121-42R" H 2400 4500 50  0001 C CNN "manf#"
 	1    2400 4500
 	-1   0    0    1
@@
 F 2 "Britishideas:TE-1871059-1" H 2400 4650 50  0001 C CNN
 F 3 "~" H 2400 4650 50  0001 C CNN
+F 4 "S7121-42R" H 2400 4650 50  0001 C CNN "manf#"
 	1    2400 4650
 	-1   0    0    1
@@
 F 2 "Britishideas:TE-1871059-1" H 2400 4800 50  0001 C CNN
 F 3 "~" H 2400 4800 50  0001 C CNN
+F 4 "S7121-42R" H 2400 4800 50  0001 C CNN "manf#"
 	1    2400 4800
 	-1   0    0    1
@@
 F 2 "Britishideas:TE-1871059-1" H 2400 4950 50  0001 C CNN
 F 3 "~" H 2400 4950 50  0001 C CNN
+F 4 "S7121-42R" H 2400 4950 50  0001 C CNN "manf#"
 	1    2400 4950
 	-1   0    0    1
@@
 F 2 "Britishideas:TE-1871059-1" H 2400 5100 50  0001 C CNN
 F 3 "~" H 2400 5100 50  0001 C CNN
+F 4 "S7121-42R" H 2400 5100 50  0001 C CNN "manf#"
 	1    2400 5100
 	-1   0    0    1
@@
 F 2 "Britishideas:TE-1871059-1" H 2400 5250 50  0001 C CNN
 F 3 "~" H 2400 5250 50  0001 C CNN
+F 4 "S7121-42R" H 2400 5250 50  0001 C CNN "manf#"
 	1    2400 5250
 	-1   0    0    1
@@
 F 2 "Britishideas:TE-1871059-1" H 2400 5400 50  0001 C CNN
 F 3 "~" H 2400 5400 50  0001 C CNN
+F 4 "S7121-42R" H 2400 5400 50  0001 C CNN "manf#"
 	1    2400 5400
 	-1   0    0    1
@@
 F 2 "Britishideas:TE-1871059-1" H 2400 5550 50  0001 C CNN
 F 3 "~" H 2400 5550 50  0001 C CNN
+F 4 "S7121-42R" H 2400 5550 50  0001 C CNN "manf#"
 	1    2400 5550
 	-1   0    0    1
@@
 F 2 "Britishideas:TE-1871059-1" H 2400 5700 50  0001 C CNN
 F 3 "~" H 2400 5700 50  0001 C CNN
+F 4 "S7121-42R" H 2400 5700 50  0001 C CNN "manf#"
 	1    2400 5700
 	-1   0    0    1
